Commit message: New, almost ready for usable simulation

File: urdf/robot_to_export.xacro (robot description, xacro)
@@ -1,7 +1,9 @@
 <?xml version="1.0" ?>
 <robot name="robot_to_export" xmlns:xacro="http://www.ros.org/wiki/xacro">
-<xacro:include filename="$(find robot_to_export_description)/urdf/materials.xacro" />
-<xacro:include filename="$(find robot_to_export_description)/urdf/robot_to_export.trans" />
-<xacro:include filename="$(find robot_to_export_description)/urdf/robot_to_export.gazebo" />
+<!-- Define materials -->
+<material name="wood">
+  <color rgba="0.588 0.435 0.200 1.000"/>
+</material>
+<!-- Define the links -->
 <link name="base_link">
   <inertial>
@@ -15,5 +17,5 @@
       <mesh filename="package://robot_to_export_description/meshes/base_link.stl" scale="0.001 0.001 0.001"/>
     </geometry>
-    <material name="silver"/>
+    <material name="wood"/>
   </visual>
   <collision>
@@ -35,5 +37,5 @@
       <mesh filename="package://robot_to_export_description/meshes/hip-thigh-joint_1.stl" scale="0.001 0.001 0.001"/>
     </geometry>
-    <material name="silver"/>
+    <material name="wood"/>
   </visual>
   <collision>
@@ -55,5 +57,5 @@
       <mesh filename="package://robot_to_export_description/meshes/thigh_1.stl" scale="0.001 0.001 0.001"/>
     </geometry>
-    <material name="silver"/>
+    <material name="wood"/>
   </visual>
   <collision>
@@ -75,5 +77,5 @@
       <mesh filename="package://robot_to_export_description/meshes/shin_1.stl" scale="0.001 0.001 0.001"/>
     </geometry>
-    <material name="silver"/>
+    <material name="wood"/>
   </visual>
   <collision>
