Commit message: Make a robot class

File: twolegged/resources/urdf/robot_to_export.xacro (robot description, xacro)
@@ -15,5 +15,5 @@
     <origin xyz="0 0 0" rpy="0 0 0"/>
     <geometry>
-      <mesh filename="package://robot_to_export_description/meshes/base_link.stl" scale="0.001 0.001 0.001"/>
+      <mesh filename="package://resources/meshes/base_link.stl" scale="0.001 0.001 0.001"/>
     </geometry>
     <material name="wood"/>
@@ -22,5 +22,5 @@
     <origin xyz="0 0 0" rpy="0 0 0"/>
     <geometry>
-      <mesh filename="package://robot_to_export_description/meshes/base_link.stl" scale="0.001 0.001 0.001"/>
+      <mesh filename="package://resources/meshes/base_link.stl" scale="0.001 0.001 0.001"/>
     </geometry>
   </collision>
@@ -35,5 +35,5 @@
     <origin xyz="-0.0696 -0.029307 0.001" rpy="0 0 0"/>
     <geometry>
-      <mesh filename="package://robot_to_export_description/meshes/hip-thigh-joint_1.stl" scale="0.001 0.001 0.001"/>
+      <mesh filename="package://resources/meshes/hip-thigh-joint_1.stl" scale="0.001 0.001 0.001"/>
     </geometry>
     <material name="wood"/>
@@ -42,5 +42,5 @@
     <origin xyz="-0.0696 -0.029307 0.001" rpy="0 0 0"/>
     <geometry>
-      <mesh filename="package://robot_to_export_description/meshes/hip-thigh-joint_1.stl" scale="0.001 0.001 0.001"/>
+      <mesh filename="package://resources/meshes/hip-thigh-joint_1.stl" scale="0.001 0.001 0.001"/>
     </geometry>
   </collision>
@@ -55,5 +55,5 @@
     <origin xyz="-0.1386 -0.029307 -0.069" rpy="0 0 0"/>
     <geometry>
-      <mesh filename="package://robot_to_export_description/meshes/thigh_1.stl" scale="0.001 0.001 0.001"/>
+      <mesh filename="package://resources/meshes/thigh_1.stl" scale="0.001 0.001 0.001"/>
     </geometry>
     <material name="wood"/>
@@ -62,5 +62,5 @@
     <origin xyz="-0.1386 -0.029307 -0.069" rpy="0 0 0"/>
     <geometry>
-      <mesh filename="package://robot_to_export_description/meshes/thigh_1.stl" scale="0.001 0.001 0.001"/>
+      <mesh filename="package://resources/meshes/thigh_1.stl" scale="0.001 0.001 0.001"/>
     </geometry>
   </collision>
@@ -75,5 +75,5 @@
     <origin xyz="-0.1586 0.560693 -0.069" rpy="0 0 0"/>
     <geometry>
-      <mesh filename="package://robot_to_export_description/meshes/shin_1.stl" scale="0.001 0.001 0.001"/>
+      <mesh filename="package://resources/meshes/shin_1.stl" scale="0.001 0.001 0.001"/>
     </geometry>
     <material name="wood"/>
@@ -82,5 +82,5 @@
     <origin xyz="-0.1586 0.560693 -0.069" rpy="0 0 0"/>
     <geometry>
-      <mesh filename="package://robot_to_export_description/meshes/shin_1.stl" scale="0.001 0.001 0.001"/>
+      <mesh filename="package://resources/meshes/shin_1.stl" scale="0.001 0.001 0.001"/>
     </geometry>
   </collision>
